Commit message: Added tf broadcaster for pan/tilt

File: catkin_ws/src/waveshare_alphabot2/urdf/Waveshare_Alphabot2.urdf (robot description, URDF)
Before this commit: robot Waveshare_Alphabot2, 13 links, 12 joints
Joints:
- removed joint camera_link
- removed joint head_pan_link
- removed joint head_tilt_link
- removed joint jointwheelLeft
- removed joint jointwheelRight
- added joint camera_joint: type fixed, parent servoTilt, child camera, origin xyz=0.0165 0.0 0.01 rpy=0 0 0
- added joint headPan_joint: type revolute, parent servoPanNeck, child servoPan, origin xyz=0.0 0.0 0.02 rpy=0 0 0, axis 0 0 1, limit lower=-1.5708 upper=1.5708 effort=100 velocity=1.0
- added joint headTilt_joint: type revolute, parent servoPan, child servoTilt, origin xyz=0.02 0.0 0.015 rpy=0 0 0, axis 0 1 0, limit lower=-1.0 upper=1.0 effort=100 velocity=1.0
- added joint wheelLeft_joint: type fixed, parent base_link, child wheelLeft, origin xyz=0.0 0.04 0.007 rpy=0 0 0, axis 0 1 0
- added joint wheelRight_joint: type fixed, parent base_link, child wheelRight, origin xyz=0.0 -0.04 0.007 rpy=0 0 0, axis 0 1 0

Commit message: Bug fixes and corrcted fiducial alignment
Small bug fixes and corrected a major issue with the fiducial alignment.

File: catkin_ws/src/waveshare_alphabot2/urdf/Waveshare_Alphabot2.urdf (robot description, URDF)
Before this commit: robot Waveshare_Alphabot2, 13 links, 12 joints
Joints:
- joint camera_joint: origin xyz=0.0165 0.0 0.01 rpy=0 0 0 -> xyz=0.0165 0.0 0.01 rpy=-1.5708 0 -1.5708
